File: source_pad/source_pad.sch (KiCad schematic (older format))
At the start: 19 parts, among them SW1 SW_PUSH, SW2 SW_PUSH, SW3 SW_PUSH, SW4 SW_PUSH, SW5 SW_PUSH, SW6 SW_PUSH, SW7 SW_PUSH, SW8 SW_PUSH, SW9 SW_PUSH, U1 ProMicro-kbd

Commit message: Updated clearances
Parts:
- U1: footprint kbd:ProMicro_v3.5 -> kbd:ProMicro_v3.5_fix
Changed lines of the file:
@@
 F 0 "U1" H 1700 3587 60  0000 C CNN
 F 1 "ProMicro-kbd" H 1700 3481 60  0000 C CNN
-F 2 "kbd:ProMicro_v3.5" H 1800 1500 60  0001 C CNN
+F 2 "kbd:ProMicro_v3.5_fix" H 1800 1500 60  0001 C CNN
 F 3 "" H 1800 1500 60  0000 C CNN
 	1    1700 2550

Commit message: fixed mx pads
Parts:
- SW1, SW2, SW3, SW4, SW5, SW6, SW7, SW8, SW9: footprint kbd:CherryMX_1u -> kbd:CherryMX_1u_fix
Changed lines of the file:
@@
 F 0 "SW2" H 4100 2055 50  0000 C CNN
 F 1 "SW_PUSH" H 4100 1964 50  0000 C CNN
-F 2 "kbd:CherryMX_1u" H 4100 1800 50  0001 C CNN
+F 2 "kbd:CherryMX_1u_fix" H 4100 1800 50  0001 C CNN
 F 3 "" H 4100 1800 50  0000 C CNN
 	1    4100 1800
@@
 F 0 "SW1" H 4100 1355 50  0000 C CNN
 F 1 "SW_PUSH" H 4100 1264 50  0000 C CNN
-F 2 "kbd:CherryMX_1u" H 4100 1100 50  0001 C CNN
+F 2 "kbd:CherryMX_1u_fix" H 4100 1100 50  0001 C CNN
 F 3 "" H 4100 1100 50  0000 C CNN
 	1    4100 1100
@@
 F 0 "SW3" H 4100 2805 50  0000 C CNN
 F 1 "SW_PUSH" H 4100 2714 50  0000 C CNN
-F 2 "kbd:CherryMX_1u" H 4100 2550 50  0001 C CNN
+F 2 "kbd:CherryMX_1u_fix" H 4100 2550 50  0001 C CNN
 F 3 "" H 4100 2550 50  0000 C CNN
 	1    4100 2550
@@
 F 0 "SW4" H 4900 1355 50  0000 C CNN
 F 1 "SW_PUSH" H 4900 1264 50  0000 C CNN
-F 2 "kbd:CherryMX_1u" H 4900 1100 50  0001 C CNN
+F 2 "kbd:CherryMX_1u_fix" H 4900 1100 50  0001 C CNN
 F 3 "" H 4900 1100 50  0000 C CNN
 	1    4900 1100
@@
 F 0 "SW7" H 5700 1355 50  0000 C CNN
 F 1 "SW_PUSH" H 5700 1264 50  0000 C CNN
-F 2 "kbd:CherryMX_1u" H 5700 1100 50  0001 C CNN
+F 2 "kbd:CherryMX_1u_fix" H 5700 1100 50  0001 C CNN
 F 3 "" H 5700 1100 50  0000 C CNN
 	1    5700 1100
@@
 F 0 "SW5" H 4900 2055 50  0000 C CNN
 F 1 "SW_PUSH" H 4900 1964 50  0000 C CNN
-F 2 "kbd:CherryMX_1u" H 4900 1800 50  0001 C CNN
+F 2 "kbd:CherryMX_1u_fix" H 4900 1800 50  0001 C CNN
 F 3 "" H 4900 1800 50  0000 C CNN
 	1    4900 1800
@@
 F 0 "SW8" H 5700 2055 50  0000 C CNN
 F 1 "SW_PUSH" H 5700 1964 50  0000 C CNN
-F 2 "kbd:CherryMX_1u" H 5700 1800 50  0001 C CNN
+F 2 "kbd:CherryMX_1u_fix" H 5700 1800 50  0001 C CNN
 F 3 "" H 5700 1800 50  0000 C CNN
 	1    5700 1800
@@
 F 0 "SW6" H 4900 2805 50  0000 C CNN
 F 1 "SW_PUSH" H 4900 2714 50  0000 C CNN
-F 2 "kbd:CherryMX_1u" H 4900 2550 50  0001 C CNN
+F 2 "kbd:CherryMX_1u_fix" H 4900 2550 50  0001 C CNN
 F 3 "" H 4900 2550 50  0000 C CNN
 	1    4900 2550
@@
 F 0 "SW9" H 5700 2805 50  0000 C CNN
 F 1 "SW_PUSH" H 5700 2714 50  0000 C CNN
-F 2 "kbd:CherryMX_1u" H 5700 2550 50  0001 C CNN
+F 2 "kbd:CherryMX_1u_fix" H 5700 2550 50  0001 C CNN
 F 3 "" H 5700 2550 50  0000 C CNN
 	1    5700 2550
